Commit message: newnew

File: rosbot_xl_description/urdf/rosbot_xl.urdf.xacro (robot description, xacro)
@@ -8,11 +8,13 @@
   <xacro:arg name="simulation_engine" default="ignition-gazebo" />
   <xacro:arg name="namespace" default="None" />
+  <xacro:arg name="controller_config_file" default="$(find rosbot_xl_controller)/config/diff_drive_controller.yaml" />
   <xacro:include filename="$(find rosbot_xl_description)/urdf/rosbot_xl_macro.urdf.xacro"
     ns="husarion" />
   <xacro:husarion.rosbot_xl_robot
-    use_sim="$(arg use_sim)"
+    controller_config_file="$(arg controller_config_file)"
     mecanum="$(arg mecanum)"
+    namespace="$(arg namespace)"
     simulation_engine="$(arg simulation_engine)"
-    namespace="$(arg namespace)" />
+    use_sim="$(arg use_sim)" />
   <xacro:include filename="$(find rosbot_xl_description)/urdf/components/antenna.urdf.xacro"
     ns="antenna" />
@@ -27,7 +29,4 @@
   <xacro:property name="lidar_xyz" value="0.12 0.0 0.0" />
   <xacro:property name="lidar_rpy" value="0.0 0.0 1.5708" />
-  <xacro:property name="lidar_use_gpu" value="true" />
-  <!-- use_gpu has to be set to true, CPU lidar doesn't work in ignition -
-    https://github.com/gazebosim/gz-sensors/issues/26 -->
   <xacro:if value="${lidar_model == 'slamtec_rplidar_s1'}">
     <xacro:include filename="$(find ros_components_description)/urdf/slamtec_rplidar_s1.urdf.xacro"
@@ -36,8 +35,5 @@
       parent_link="${lidar_parent_link}"
       xyz="${lidar_xyz}"
-      rpy="${lidar_rpy}"
-      use_gpu="${lidar_use_gpu}"
-      simulation_engine="$(arg simulation_engine)"
-      namespace="$(arg namespace)" />
+      rpy="${lidar_rpy}" />
   </xacro:if>
   <xacro:if value="${lidar_model == 'slamtec_rplidar_s2'}">
@@ -47,8 +43,5 @@
       parent_link="${lidar_parent_link}"
       xyz="${lidar_xyz}"
-      rpy="${lidar_rpy}"
-      use_gpu="${lidar_use_gpu}"
-      simulation_engine="$(arg simulation_engine)"
-      namespace="$(arg namespace)" />
+      rpy="${lidar_rpy}" />
   </xacro:if>
   <xacro:if value="${lidar_model == 'slamtec_rplidar_s3'}">
@@ -58,8 +51,5 @@
       parent_link="${lidar_parent_link}"
       xyz="${lidar_xyz}"
-      rpy="${lidar_rpy}"
-      use_gpu="${lidar_use_gpu}"
-      simulation_engine="$(arg simulation_engine)"
-      namespace="$(arg namespace)" />
+      rpy="${lidar_rpy}" />
   </xacro:if>
   <xacro:if value="${lidar_model == 'slamtec_rplidar_a2'}">
@@ -69,8 +59,5 @@
       parent_link="${lidar_parent_link}"
       xyz="${lidar_xyz}"
-      rpy="${lidar_rpy}"
-      use_gpu="${lidar_use_gpu}"
-      simulation_engine="$(arg simulation_engine)"
-      namespace="$(arg namespace)" />
+      rpy="${lidar_rpy}" />
   </xacro:if>
   <xacro:if value="${lidar_model == 'slamtec_rplidar_a3'}">
@@ -80,8 +67,5 @@
       parent_link="${lidar_parent_link}"
       xyz="${lidar_xyz}"
-      rpy="${lidar_rpy}"
-      use_gpu="${lidar_use_gpu}"
-      simulation_engine="$(arg simulation_engine)"
-      namespace="$(arg namespace)" />
+      rpy="${lidar_rpy}" />
   </xacro:if>
   <xacro:if value="${lidar_model == 'velodyne_puck'}">
@@ -91,9 +75,5 @@
       parent_link="${lidar_parent_link}"
       xyz="${lidar_xyz}"
-      rpy="${lidar_rpy}"
-      use_gpu="${lidar_use_gpu}"
-      simulation_engine="$(arg simulation_engine)"
-      topic="velodyne_points"
-      namespace="$(arg namespace)" />
+      rpy="${lidar_rpy}" />
   </xacro:if>
   <!-- INCLUDE CAMERA -->
@@ -112,7 +92,5 @@
       xyz="${camera_xyz}"
       rpy="${camera_rpy}"
-      use_nominal_extrinsics="$(arg use_sim)"
-      simulation_engine="$(arg simulation_engine)"
-      namespace="$(arg namespace)" />
+      use_nominal_extrinsics="$(arg use_sim)" />
   </xacro:if>
   <xacro:if value="${camera_model == 'orbbec_astra'}">
@@ -123,7 +101,5 @@
       parent_link="${camera_parent_link}"
       xyz="${camera_xyz}"
-      rpy="${camera_rpy}"
-      simulation_engine="$(arg simulation_engine)"
-      namespace="$(arg namespace)" />
+      rpy="${camera_rpy}" />
   </xacro:if>
   <xacro:if value="${camera_model.startswith('stereolabs')}">
@@ -153,7 +129,5 @@
       xyz="${camera_xyz}"
       rpy="${camera_rpy}"
-      model="${camera_model_type}"
-      simulation_engine="$(arg simulation_engine)"
-      namespace="$(arg namespace)" />
+      model="${camera_model_type}" />
   </xacro:if>
   <!-- INCLUDE CAMERA MOUNT - add if camera_model is not empty -->
